Commit message: made it fully working

File: urdf/common/castor.xacro (robot description, xacro)
@@ -10,7 +10,5 @@
                     <sphere radius="${castor_wheel_radius}" />
                 </geometry>
-                <material name="gray">
-                    <color rgba="0.3 0.3 0.3 1.0" />
-                </material>
+                <material name="Grey"/>
             </visual>
             <collision>
@@ -23,12 +21,16 @@
         </link>
         <joint name="${name}_joint" type="fixed">
-            <parent link="chassis_link" />
+            <parent link="base_link" />
             <child link="${name}_link" />
             <origin xyz="${wheel_end_sign * (chassis_length / x_divide)} ${wheel_side_sign * (chassis_width / y_divide)} ${- (chassis_height / 2.0)}" rpy="0 0 0" />
         </joint>
-        <gazebo reference="front_caster">
+        <gazebo reference="${name}_link">
             <material>Gazebo/Grey</material>
-            <mu1 value="0.001" />
-            <mu2 value="0.001" />
+            <mu1>0.1</mu1>
+            <mu2>0.1</mu2>
+            <kp>100000.0</kp>
+            <kd>10.0</kd>
+            <minDepth>0.001</minDepth>
+            <maxVel>0.1</maxVel>
         </gazebo>
     </xacro:macro>

File: urdf/common/chassis.xacro (robot description, xacro)
@@ -5,17 +5,10 @@
         <link name="base_footprint" />
         <!-- Robot Footprint -->
-        <link name="base_link" />
-        <joint name="base_joint" type="fixed">
-            <parent link="base_footprint" />
-            <child link="base_link" />
-            <origin xyz="0.0 0.0 ${chassis_ground_clearance + chassis_height / 2}" rpy="0 0 0" />
-        </joint>
-        <!-- Chassis -->
-        <link name="chassis_link">
+        <link name="base_link">
             <visual>
                 <geometry>
                     <box size="${chassis_length} ${chassis_width} ${chassis_height}" />
                 </geometry>
-                <material name="Cyan"/>
+                <material name="Turquoise"/>
             </visual>
             <collision>
@@ -26,9 +19,12 @@
             <xacro:box_inertia mass="${chassis_mass}" width="${chassis_width}" length="${chassis_length}" height="${chassis_height}" />
         </link>
-        <joint name="chassis_joint" type="fixed">
+        <joint name="base_joint" type="fixed">
             <parent link="base_link" />
-            <child link="chassis_link" />
-            <origin xyz="0.0 0.0 0.0" rpy="0 0 0" />
+            <child link="base_footprint" />
+            <origin xyz="0.0 0.0 -${chassis_ground_clearance + chassis_height / 2}" rpy="0 0 0" />
         </joint>
+        <gazebo reference="base_link">
+            <material>Gazebo/Turquoise</material>
+        </gazebo>
     </xacro:macro>
 </robot>

File: urdf/common/materials.xacro (robot description, xacro)
@@ -14,5 +14,8 @@
     <color rgba="1 1 0 1"/>
   </material>
-  <material name="Cyan">
+  <material name="Orange">
+    <color rgba="1 0.647 0 1"/>
+  </material>
+  <material name="Turquoise">
     <color rgba="0 1 1 1"/>
   </material>

File: urdf/common/wheel.xacro (robot description, xacro)
@@ -11,5 +11,5 @@
                     <cylinder radius="${wheel_radius}" length="${wheel_width}" />
                 </geometry>
-                <material name="Grey"/>
+                <material name="Orange"/>
             </visual>
             <collision>
@@ -22,20 +22,19 @@
         </link>
         <joint name="${name}_joint" type="continuous">
-            <parent link="chassis_link" />
+            <parent link="base_link" />
             <child link="${name}_link" />
             <origin
-                xyz="0.0 ${(wheel_side_sign * (chassis_width + wheel_width + wheel_gap)) / 2.0} 0.0"
+                xyz="0.0 ${(wheel_side_sign * (chassis_width + wheel_width + wheel_gap)) / 2.0} ${wheel_radius - (chassis_ground_clearance + chassis_height / 2.0)}"
                 rpy="0 0 0" />
             <axis xyz="0 1 0" />
         </joint>
         <gazebo reference="${name}_link">
-            <material>Gazebo/Grey</material>
-            <mu1>1000000000000000.0</mu1>
-            <mu2>1000000000000000.0</mu2>
-            <kp>1000000000000.0</kp>
+            <material>Gazebo/Orange</material>
+            <mu1>1.0</mu1>
+            <mu2>1.0</mu2>
+            <kp>100000.0</kp>
             <kd>10.0</kd>
             <minDepth>0.001</minDepth>
             <maxVel>0.1</maxVel>
-            <fdir1>1 0 0</fdir1>
         </gazebo>
     </xacro:macro>

File: urdf/properties.xacro (robot description, xacro)
@@ -10,5 +10,5 @@
         <xacro:property name="chassis_ground_clearance" value="0.05" />
         <!-- Wheels -->
-        <xacro:property name="wheel_radius" value="${(chassis_height / 2.0) + chassis_ground_clearance}"/>
+        <xacro:property name="wheel_radius" value="${(chassis_height / 3.0) + chassis_ground_clearance}"/>
         <xacro:property name="wheel_width" value="0.05" />
         <xacro:property name="wheel_mass" value="0.1" />
@@ -17,8 +17,12 @@
         <xacro:property name="castor_wheel_radius" value="${chassis_ground_clearance}"/>
         <xacro:property name="castor_mass" value="0.1"/>
+        <!-- Diff Drive -->
+         <xacro:property name="publish_odom_tf" value="true"/>
         <!-- Lidar -->
         <xacro:property name="lidar_width" value="0.0508"/>
         <xacro:property name="lidar_thickness" value="0.055"/>
         <xacro:property name="lidar_mass" value="0.125"/>
+        <xacro:property name="visualize_lidar" value="false">
+        </xacro:property>
     </xacro:if>
 </robot>

File: urdf/robot.urdf.xacro (robot description, xacro)
@@ -16,4 +16,6 @@
     <!-- Sensors -->
     <xacro:include filename="$(find questbot_description)/urdf/sensors/sensors.xacro"/>
+    <!-- Drives -->
+    <xacro:include filename="$(find questbot_description)/urdf/drives/drives.xacro"/>
     <!-- Chassis -->
     <xacro:chassis />
@@ -21,11 +23,13 @@
     <xacro:if value="$(arg use_2wd)">
         <!-- Wheels -->
-        <xacro:wheel name="left_wheel" wheel_side_sign="-1"/>
-        <xacro:wheel name="right_wheel" wheel_side_sign="1"/>
+        <xacro:wheel name="left_wheel" wheel_side_sign="1"/>
+        <xacro:wheel name="right_wheel" wheel_side_sign="-1"/>
+        <!-- Diff Drive -->
+        <xacro:diffdrive left_wheel_name="left_wheel" right_wheel_name="right_wheel"/>
         <!-- Castors -->
-        <xacro:castor_wheel name="front_left_castor_wheel"  x_divide="3.0" wheel_end_sign="1" y_divide="4.0" wheel_side_sign="-1"/>
-        <xacro:castor_wheel name="front_right_castor_wheel"  x_divide="3.0" wheel_end_sign="1" y_divide="4.0" wheel_side_sign="1"/>
-        <xacro:castor_wheel name="back_left_castor_wheel"  x_divide="3.0" wheel_end_sign="-1" y_divide="4.0" wheel_side_sign="-1"/>
-        <xacro:castor_wheel name="back_right_castor_wheel"  x_divide="3.0" wheel_end_sign="-1" y_divide="4.0" wheel_side_sign="1"/>
+        <xacro:castor_wheel name="front_left_castor_wheel"  x_divide="3.0" wheel_end_sign="1" y_divide="4.0" wheel_side_sign="1"/>
+        <xacro:castor_wheel name="front_right_castor_wheel"  x_divide="3.0" wheel_end_sign="1" y_divide="4.0" wheel_side_sign="-1"/>
+        <xacro:castor_wheel name="back_left_castor_wheel"  x_divide="3.0" wheel_end_sign="-1" y_divide="4.0" wheel_side_sign="1"/>
+        <xacro:castor_wheel name="back_right_castor_wheel"  x_divide="3.0" wheel_end_sign="-1" y_divide="4.0" wheel_side_sign="-1"/>
         <!-- Lidar -->
          <xacro:lidar name="lidar" x="0.0" y="0.0" z="${(chassis_height + lidar_thickness) / 2.0}" />

File: urdf/sensors/lidar.xacro (robot description, xacro)
@@ -8,7 +8,5 @@
                     <cylinder radius="${lidar_width}" length="${lidar_thickness}" />
                 </geometry>
-                <material name="green">
-                    <color rgba="0.0 1.0 0.0 1.0" />
-                </material>
+                <material name="Green"/>
             </visual>
             <collision>
@@ -21,5 +19,5 @@
         </link>
         <joint name="${name}_joint" type="fixed">
-            <parent link="chassis_link" />
+            <parent link="base_link" />
             <child link="${name}_link" />
             <origin xyz="${x} ${y} ${z}" rpy="0 0 0" />
@@ -29,5 +27,5 @@
             <sensor name="lidar" type="ray">
                 <always_on>true</always_on>
-                <visualize>true</visualize>
+                <visualize>${visualize_lidar}</visualize>
                 <update_rate>5</update_rate>
                 <ray>
