Commit message: minor improvements

File: urdf/drives/diffdrive.xacro (robot description, xacro)
@@ -10,4 +10,5 @@
                 <wheel_separation>${chassis_width + wheel_gap}</wheel_separation>
                 <wheel_radius>${wheel_radius}</wheel_radius>
+                <wheel_diameter>${wheel_radius * 2}</wheel_diameter>
                 <!-- limits -->
                 <max_wheel_torque>20</max_wheel_torque>

File: urdf/properties.xacro (robot description, xacro)
@@ -23,6 +23,7 @@
         <xacro:property name="lidar_thickness" value="0.055"/>
         <xacro:property name="lidar_mass" value="0.125"/>
-        <xacro:property name="visualize_lidar" value="false">
-        </xacro:property>
+        <xacro:property name="visualize_lidar" value="true"/>
+        <xacro:property name="lidar_min_range" value="0.12"/>
+        <xacro:property name="lidar_max_range" value="30.0"/>
     </xacro:if>
 </robot>

File: urdf/sensors/lidar.xacro (robot description, xacro)
@@ -39,13 +39,8 @@
                     </scan>
                     <range>
-                        <min>0.120000</min>
-                        <max>3.5</max>
+                        <min>${lidar_min_range}</min>
+                        <max>${lidar_max_range}</max>
                         <resolution>0.015000</resolution>
                     </range>
-                    <noise>
-                        <type>gaussian</type>
-                        <mean>0.0</mean>
-                        <stddev>0.01</stddev>
-                    </noise>
                 </ray>
                 <plugin name="scan" filename="libgazebo_ros_ray_sensor.so">
