Commit message: added lidar

File: urdf/properties.xacro (robot description, xacro)
@@ -17,4 +17,8 @@
         <xacro:property name="castor_wheel_radius" value="${chassis_ground_clearance}"/>
         <xacro:property name="castor_mass" value="0.1"/>
+        <!-- Lidar -->
+        <xacro:property name="lidar_width" value="0.0508"/>
+        <xacro:property name="lidar_thickness" value="0.055"/>
+        <xacro:property name="lidar_mass" value="0.125"/>
     </xacro:if>
 </robot>

File: urdf/robot.urdf.xacro (robot description, xacro)
@@ -14,4 +14,6 @@
     <!-- Castor Wheel -->
     <xacro:include filename="$(find questbot_description)/urdf/common/castor.xacro"/>
+    <!-- Sensors -->
+    <xacro:include filename="$(find questbot_description)/urdf/sensors/sensors.xacro"/>
     <!-- Chassis -->
     <xacro:chassis />
@@ -26,4 +28,6 @@
         <xacro:castor_wheel name="back_left_castor_wheel"  x_divide="3.0" wheel_end_sign="-1" y_divide="4.0" wheel_side_sign="-1"/>
         <xacro:castor_wheel name="back_right_castor_wheel"  x_divide="3.0" wheel_end_sign="-1" y_divide="4.0" wheel_side_sign="1"/>
+        <!-- Lidar -->
+         <xacro:lidar name="lidar" x="0.0" y="0.0" z="${(chassis_height + lidar_thickness) / 2.0}" />
     </xacro:if>
 </robot>

Commit message: turned of lidar viz

File: urdf/properties.xacro (robot description, xacro)
@@ -23,5 +23,5 @@
         <xacro:property name="lidar_thickness" value="0.055"/>
         <xacro:property name="lidar_mass" value="0.125"/>
-        <xacro:property name="visualize_lidar" value="true"/>
+        <xacro:property name="visualize_lidar" value="false"/>
         <xacro:property name="lidar_min_range" value="0.12"/>
         <xacro:property name="lidar_max_range" value="30.0"/>
